File: ECAM/Bed of Nails ISSUE_PROTO_B/Power.sch (KiCad schematic (older format))
At the start: 33 parts, among them Q1 MGSF1N02L, Q2 MGSF1N02L, U1 TPS62850x-Q1, U2 TPS62850x-Q1, U3 LTC4353

Commit message: set up test points for TSM570 schematic
Parts:
- removed C1, C16, C6, C7: 100n-10V-0402-5%-CER, TFT_C_passive_SMD:0402_CAP, symbol TFT_capacitors:100n-10V-0402-5%-CER
- removed C10, C11, C12, C13: 10u-10V-0603-10%-CER, TFT_C_passive_SMD:1206_CAP_TANT, symbol TFT_capacitors:10u-10V-0603-10%-CER
- removed C14, C15: 56n-16V-0402-10%-CER, TFT_C_passive_SMD:0402_CAP, symbol TFT_capacitors:56n-16V-0402-10%-CER
- removed C2, C3: 1u-10V-0603-10%-CER, TFT_C_passive_SMD:0603_CAP, symbol TFT_capacitors:1u-10V-0603-10%-CER
- removed C4, C5: 10u-10V-1206-10%-TANT, TFT_C_passive_SMD:1206_CAP_TANT, symbol TFT_capacitors:10u-10V-1206-10%-TANT
- removed C8, C9: 10p-50V-0402-0.5p-CER, TFT_C_passive_SMD:0402_CAP, symbol TFT_capacitors:10p-50V-0402-0.5p-CER
- removed L1, L2: 470nH-4A-20%, TFT_I_passive_SMD:2.5x2mm_I_SMD, symbol TFT_inductors:470nH-4A-20%
- removed Q1, Q2: MGSF1N02L, Package_TO_SOT_SMD:SOT-23, symbol TFT_semiconductors:MGSF1N02L
- removed R1, R2: 100K-50V-0402-1%, TFT_R_passive_SMD:0402_RES, symbol TFT_resistors:100K-50V-0402-1%
- removed R3, R5: 16K2-50V-0402-1%, TFT_R_passive_SMD:0402_RES, symbol TFT_resistors:16K2-50V-0402-1%
- removed R4, R6: 15K-50V-0402-1%, TFT_R_passive_SMD:0402_RES, symbol TFT_resistors:15K-50V-0402-1%
- removed TP16, TP19: TEST-POINT, TFT_TestPoints:TP_RDPad_D1.0mm, symbol TFT_testpoints:TEST-POINT
- removed U1, U2: TPS62850x-Q1, TFT_SOT:SOT-583, symbol TFT_SMPS:TPS62850x-Q1
- removed U3: LTC4353, Package_DFN_QFN:DFN-16-1EP_3x4mm_P0.45mm_EP1.7x3.3mm, symbol TFT_drivers:LTC4353
- added TP? (x3): TEST-POINT, TFT_TestPoints:TP_RDPad_D1.0mm, symbol TFT_testpoints:TEST-POINT
Connections:
- net labels removed: GATE_1, GATE_2, GND, OBC_3V3
- wire segments 157 -> 5
Other:
- note removed: "Bulk decoupling"
- moved on the sheet: TP17, TP18
