File: ECAM/Bed of Nails ISSUE_PROTO_B/Connectors.sch (KiCad schematic (older format))
At the start: 2 parts, among them J1 ERM8-020-X, J2 ERF6-020-X

Commit message: updated RFC connector on BoN to ERF8 for bottom layer mounting
Parts:
- removed J1: ERM8-020-X, TFT_connectors:ERM8-020-XX.X-X-DV, symbol TFT_connectors:ERM8-020-X
- removed J2: ERF6-020-X, TFT_connectors:ERF6-020-XX.X-X-DV-A-XX-K, symbol TFT_connectors:ERF6-020-X
- added J1: ERF8-020-X, TFT_connectors:ERF8-020-XX.X-X-DV, symbol TFT_connectors:ERF8-020-X
Connections:
- wire segments 142 -> 66
Other:
- note removed: "Payload Connector"
