File: ECAM/Bed of Nails ISSUE_PROTO_B/TMS570_uC.sch (KiCad schematic (older format))
At the start: 33 parts, among them U11 TMS5701227CZWTQQ1, X2 LFTCXO075797

Commit message: set up test points for TSM570 schematic
Parts:
- removed C28, C29: 1u-10V-0603-10%-CER, TFT_C_passive_SMD:0603_CAP, symbol TFT_capacitors:1u-10V-0603-10%-CER
- removed C30, C31, C32, C33, C34, C35, C36, C37, C38, C39, C40, C41, C42: 100n-10V-0402-5%-CER, TFT_C_passive_SMD:0402_CAP, symbol TFT_capacitors:100n-10V-0402-5%-CER
- removed R17, R18, R19, R20: 4K7-50V-0402-1%, TFT_R_passive_SMD:0402_RES, symbol TFT_resistors:4K7-50V-0402-1%
- removed R23, R24: 0R-50V-0402, TFT_R_passive_SMD:0402_RES, symbol TFT_resistors:0R-50V-0402
- removed U11: TMS5701227CZWTQQ1, TFT_BGA:ZWT337, symbol TFT_uC:TMS5701227CZWTQQ1
- removed X2: LFTCXO075797, TFT_XTAL:LFTCXO075797, symbol TFT_oscillators:LFTCXO075797
Connections:
- net labels removed: ADS_nRST, CAN_PA_Rs, CAN_PL_Rs, CAN_R_Rs, FL_1_CLK, FL_1_SI_IO0, FL_1_SO_IO1, FL_1_nCS1, FL_1_nCS2, FL_1_nHOLD_IO3, FL_1_nRESET, FRAM_1_CIPO, FRAM_1_CLK, FRAM_1_COPI, FRAM_1_nCS, GND, GPS_P1PPS, GPS_RXD0, GPS_STS, GPS_TXD0, GPS_nRST, JTAG_RTCK, JTAG_TCK, JTAG_TDI, JTAG_TDO, JTAG_TEST, JTAG_TMS, JTAG_nTRST, OBC_1V25, OBC_1V25_P_PG, OBC_1V25_R_PG, OBC_3V3, RTC_CLKOUT, RTC_nINT, SPVSR_PET, uC_OSC_IN
- wire segments 463 -> 10
Other:
- note added: "CAN"
- note added: "Hard reset pin"
- note added: "I2C bus"
- note added: "PORRST pin"
- note removed: "Can select GPIO or EXTCLKIN2\nfor RTC CLKOUT"
- note removed: "DNF"
- note removed: "Decoupling"
- note removed: "Temperature Compensated \nCrystal Oscillator"
- note removed: "Test + debug interface"
- moved on the sheet: TP20, TP21, TP22, TP23, TP24, TP25, TP26, TP27, TP28, TP29
