File: ECAM/Singularity ISSUE_PROTO_B_v04/OBC-1.kicad_pcb (KiCad board)
At the start: 6 copper layers, 42.8 x 42.8 mm, 121 parts, among them J1 ERM8-020-X, J2 ERF6-020-X, Q1 MGSF1N02L, Q2 MGSF1N02L, U1 TPS62850x-Q1, U10 RV-3032-C7, U11 TMS5701227CZWTQQ1, U12 TMP100, U2 TPS62850x-Q1, U3 LTC4353, U4 SN65HVD230M-EP, U5 SN65HVD230M-EP, U6 SN65HVD230M-EP, U7 CY15B108QI, U8 S70FL01GS, U9 TPS3813K33-EP, X2 LFTCXO075797

Commit message: migrated to KiCAD v6.  For now, old v5 files remain as legacy.  Please only use v6 from now on
Routing:
- added copper zone on In1.Cu, net GND
- added copper zone on In4.Cu, net GND
- removed copper zone on In1_GND.Cu, net GND
- removed copper zone on In4_GND.Cu, net GND
Other:
- net class Default removed
